Commit message: add lunar world, camera to gazebo model, and camera inspect poses

File: canadarm2/canadarm_description/models/urdf/SSRMS_Canadarm2.gazebo.xacro (robot description, xacro)
@@ -56,4 +56,25 @@
             </plugin>
         </gazebo>
+        <gazebo reference="ee_camera">
+            <sensor type="camera" name="camera_sensor">
+                <pose>0 0 0 3.14 0 0</pose>
+                <visualize>1</visualize>
+                <update_rate>10.0</update_rate>
+                <camera>
+                    <!-- <horizontal_fov>1.3962634</horizontal_fov> -->
+                    <image>
+                        <width>800</width>
+                        <height>800</height>
+                        <format>R8G8B8</format>
+                    </image>
+                    <noise>
+                    <type>gaussian</type>
+                    <stddev>0.007</stddev>
+                    </noise>
+                </camera>
+                <always_on>1</always_on>
+                <topic>image_raw</topic>
+            </sensor>
+        </gazebo>
         <!-- Colors -->
         <material name="White">

File: canadarm2/canadarm_description/models/urdf/SSRMS_Canadarm2.urdf.xacro (robot description, xacro)
@@ -290,3 +290,13 @@
     </collision>
   </link>
+  <!-- Joint 7: Wrist Roll Joint -->
+  <joint name="ee_to_camera" type="fixed">
+    <parent link="EE_SSRMS"/>
+    <child link="ee_camera"/>
+    <origin rpy="0 1.570 0" xyz="-0.30 0.0 -1.15"/>
+    <axis xyz="0 0 1"/>
+    <limit lower="0" upper="0" effort="0" velocity="0"/>
+  </joint>
+  <!-- camera link -->
+  <link name="ee_camera"/>
 </robot>

Commit message: Update Canadarm demo for Jazzy (#82).
Update Canadarm demo to work with ROS 2 Jazzy and Gazebo Harmonic.

Co-authored-by: Ana Huaman <ana@traclabs.com>

File: canadarm2/canadarm_description/models/urdf/SSRMS_Canadarm2.gazebo.xacro (robot description, xacro)
@@ -2,7 +2,7 @@
 <robot xmlns:xacro="http://wiki.ros.org/xacro">
     <xacro:macro name="ssrms_canadarm2_gazebo" params="command_interface:=effort">
-        <ros2_control name="IgnitionSystem" type="system">
+        <ros2_control name="GazeboSystem" type="system">
             <hardware>
-                <plugin>ign_ros2_control/IgnitionSystem</plugin>
+                <plugin>gz_ros2_control/GazeboSimSystem</plugin>
             </hardware>
             <joint name="Base_Joint">
@@ -50,5 +50,5 @@
         </ros2_control>
         <gazebo>
-            <plugin filename="libign_ros2_control-system" name="ign_ros2_control::IgnitionROS2ControlPlugin">
+            <plugin filename="gz_ros2_control-system" name="gz_ros2_control::GazeboSimROS2ControlPlugin">
                 <robot_param>robot_description</robot_param>
                 <robot_param_node>robot_state_publisher</robot_param_node>

File: canadarm2/canadarm_description/models/urdf/SSRMS_Canadarm2.urdf.xacro (robot description, xacro)
@@ -28,5 +28,5 @@
       <origin rpy="0 0 0" xyz="0 0 0"/>
       <geometry>
-        <mesh filename="$(find canadarm_description)/models/meshes/ee.dae" scale="1.0 1.0 1.0" />
+        <mesh filename="file://$(find canadarm_description)/models/meshes/ee.dae" scale="1.0 1.0 1.0" />
       </geometry>
     </visual>
@@ -34,5 +34,5 @@
       <origin rpy="0 0 0" xyz="0 0 0"/>
       <geometry>
-        <mesh filename="$(find canadarm_description)/models/meshes/ee.stl" scale="1.0 1.0 1.0" />
+        <mesh filename="file://$(find canadarm_description)/models/meshes/ee.stl" scale="1.0 1.0 1.0" />
       </geometry>
     </collision>
@@ -58,11 +58,11 @@
       <origin rpy="0 -1.5708 0" xyz="0.25082 0 -0.175"/>
       <geometry>
-        <mesh filename="$(find canadarm_description)/models/meshes/joint_v3_0.dae" scale="1.0 1.0 1.0" />
-      </geometry>
-    </visual>
-    <collision>
-      <origin rpy="0 -1.5708 0" xyz="0.25082 0 -0.175"/>
-      <geometry>
-        <mesh filename="$(find canadarm_description)/models/meshes/joint_v3_0.stl" scale="1.0 1.0 1.0" />
+        <mesh filename="file://$(find canadarm_description)/models/meshes/joint_v3_0.dae" scale="1.0 1.0 1.0" />
+      </geometry>
+    </visual>
+    <collision>
+      <origin rpy="0 -1.5708 0" xyz="0.25082 0 -0.175"/>
+      <geometry>
+        <mesh filename="file://$(find canadarm_description)/models/meshes/joint_v3_0.stl" scale="1.0 1.0 1.0" />
       </geometry>
     </collision>
@@ -86,5 +86,5 @@
       <origin rpy="0 0 0" xyz="0.175 0 -0.25082"/>
       <geometry>
-        <mesh filename="$(find canadarm_description)/models/meshes/joint_v3_0.dae" scale="1.0 1.0 1.0" />
+        <mesh filename="file://$(find canadarm_description)/models/meshes/joint_v3_0.dae" scale="1.0 1.0 1.0" />
       </geometry>
     </visual>
@@ -92,5 +92,5 @@
       <origin rpy="0 0 0" xyz="0.175 0 -0.25082"/>
       <geometry>
-        <mesh filename="$(find canadarm_description)/models/meshes/joint_v3_0.stl" scale="1.0 1.0 1.0" />
+        <mesh filename="file://$(find canadarm_description)/models/meshes/joint_v3_0.stl" scale="1.0 1.0 1.0" />
       </geometry>
     </collision>
@@ -114,11 +114,11 @@
       <origin rpy="0 -1.5708 0" xyz="0.25082 0 -0.175"/>
       <geometry>
-        <mesh filename="$(find canadarm_description)/models/meshes/joint_v3_0.dae" scale="1.0 1.0 1.0" />
-      </geometry>
-    </visual>
-    <collision>
-      <origin rpy="0 -1.5708 0" xyz="0.25082 0 -0.175"/>
-      <geometry>
-        <mesh filename="$(find canadarm_description)/models/meshes/joint_v3_0.stl" scale="1.0 1.0 1.0" />
+        <mesh filename="file://$(find canadarm_description)/models/meshes/joint_v3_0.dae" scale="1.0 1.0 1.0" />
+      </geometry>
+    </visual>
+    <collision>
+      <origin rpy="0 -1.5708 0" xyz="0.25082 0 -0.175"/>
+      <geometry>
+        <mesh filename="file://$(find canadarm_description)/models/meshes/joint_v3_0.stl" scale="1.0 1.0 1.0" />
       </geometry>
     </collision>
@@ -126,5 +126,5 @@
       <origin rpy="-1.5708 0 -1.5708" xyz="0.25082 0 -0.175"/>
       <geometry>
-        <mesh filename="$(find canadarm_description)/models/meshes/long_link_1_v3_0.dae" scale="1.0 1.0 1.0" />
+        <mesh filename="file://$(find canadarm_description)/models/meshes/long_link_1_v3_0.dae" scale="1.0 1.0 1.0" />
       </geometry>
     </visual>
@@ -132,5 +132,5 @@
       <origin rpy="-1.5708 0 -1.5708" xyz="0.25082 0 -0.175"/>
       <geometry>
-        <mesh filename="$(find canadarm_description)/models/meshes/long_link_1_v3_0.stl" scale="1.0 1.0 1.0" />
+        <mesh filename="file://$(find canadarm_description)/models/meshes/long_link_1_v3_0.stl" scale="1.0 1.0 1.0" />
       </geometry>
     </collision>
@@ -138,5 +138,5 @@
       <origin rpy="0 1.5708 0" xyz="7.36082 0 -0.175"/>
       <geometry>
-        <mesh filename="$(find canadarm_description)/models/meshes/joint_v3_0.dae" scale="1.0 1.0 1.0" />
+        <mesh filename="file://$(find canadarm_description)/models/meshes/joint_v3_0.dae" scale="1.0 1.0 1.0" />
       </geometry>
     </visual>
@@ -144,5 +144,5 @@
       <origin rpy="0 1.5708 0" xyz="7.36082 0 -0.175"/>
       <geometry>
-        <mesh filename="$(find canadarm_description)/models/meshes/joint_v3_0.stl" scale="1.0 1.0 1.0" />
+        <mesh filename="file://$(find canadarm_description)/models/meshes/joint_v3_0.stl" scale="1.0 1.0 1.0" />
       </geometry>
     </collision>
@@ -172,5 +172,5 @@
       <origin rpy="0 1.5708 0" xyz="-0.25082 0 -0.175"/>
       <geometry>
-        <mesh filename="$(find canadarm_description)/models/meshes/link_joint_v2_1.dae" scale="1.0 1.0 1.0" />
+        <mesh filename="file://$(find canadarm_description)/models/meshes/link_joint_v2_1.dae" scale="1.0 1.0 1.0" />
       </geometry>
     </visual>
@@ -178,5 +178,5 @@
       <origin rpy="0 1.5708 0" xyz="-0.25082 0 -0.175"/>
       <geometry>
-        <mesh filename="$(find canadarm_description)/models/meshes/link_joint_v2_1.stl" scale="1.0 1.0 1.0" />
+        <mesh filename="file://$(find canadarm_description)/models/meshes/link_joint_v2_1.stl" scale="1.0 1.0 1.0" />
       </geometry>
     </collision>
@@ -184,5 +184,5 @@
       <origin rpy="1.57 -3.14 1.57" xyz="-7.36082 0 -0.175"/>
       <geometry>
-        <mesh filename="$(find canadarm_description)/models/meshes/long_link_2_v3_0.dae" scale="1.0 1.0 1.0" />
+        <mesh filename="file://$(find canadarm_description)/models/meshes/long_link_2_v3_0.dae" scale="1.0 1.0 1.0" />
       </geometry>
     </visual>
@@ -190,5 +190,5 @@
       <origin rpy="1.57 -3.14 1.57" xyz="-7.36082 0 -0.175"/>
       <geometry>
-        <mesh filename="$(find canadarm_description)/models/meshes/long_link_2_v3_0.stl" scale="1.0 1.0 1.0" />
+        <mesh filename="file://$(find canadarm_description)/models/meshes/long_link_2_v3_0.stl" scale="1.0 1.0 1.0" />
       </geometry>
     </collision>
@@ -196,5 +196,5 @@
       <origin rpy="0 -1.57 0" xyz="-7.36082 0 -0.175"/>
       <geometry>
-        <mesh filename="$(find canadarm_description)/models/meshes/joint_v3_0.dae" scale="1.0 1.0 1.0" />
+        <mesh filename="file://$(find canadarm_description)/models/meshes/joint_v3_0.dae" scale="1.0 1.0 1.0" />
       </geometry>
     </visual>
@@ -202,5 +202,5 @@
       <origin rpy="0 -1.57 0" xyz="-7.36082 0 -0.175"/>
       <geometry>
-        <mesh filename="$(find canadarm_description)/models/meshes/joint_v3_0.stl" scale="1.0 1.0 1.0" />
+        <mesh filename="file://$(find canadarm_description)/models/meshes/joint_v3_0.stl" scale="1.0 1.0 1.0" />
       </geometry>
     </collision>
@@ -224,5 +224,5 @@
       <origin rpy="0 -3.14 0" xyz="0 0 0"/>
       <geometry>
-        <mesh filename="$(find canadarm_description)/models/meshes/joint_v3_0.dae" scale="1.0 1.0 1.0" />
+        <mesh filename="file://$(find canadarm_description)/models/meshes/joint_v3_0.dae" scale="1.0 1.0 1.0" />
       </geometry>
     </visual>
@@ -230,5 +230,5 @@
       <origin rpy="0 -3.14 0" xyz="0 0 0"/>
       <geometry>
-        <mesh filename="$(find canadarm_description)/models/meshes/joint_v3_0.stl" scale="1.0 1.0 1.0" />
+        <mesh filename="file://$(find canadarm_description)/models/meshes/joint_v3_0.stl" scale="1.0 1.0 1.0" />
       </geometry>
     </collision>
@@ -252,5 +252,5 @@
       <origin rpy="0 -1.5708 0" xyz="0 0 0"/>
       <geometry>
-        <mesh filename="$(find canadarm_description)/models/meshes/joint_v3_0.dae" scale="1.0 1.0 1.0" />
+        <mesh filename="file://$(find canadarm_description)/models/meshes/joint_v3_0.dae" scale="1.0 1.0 1.0" />
       </geometry>
     </visual>
@@ -258,5 +258,5 @@
       <origin rpy="0 -1.5708 0" xyz="0 0 0"/>
       <geometry>
-        <mesh filename="$(find canadarm_description)/models/meshes/joint_v3_0.stl" scale="1.0 1.0 1.0" />
+        <mesh filename="file://$(find canadarm_description)/models/meshes/joint_v3_0.stl" scale="1.0 1.0 1.0" />
       </geometry>
     </collision>
@@ -280,5 +280,5 @@
       <origin rpy="0 -3.1415 0" xyz="0 0 0"/>
       <geometry>
-        <mesh filename="$(find canadarm_description)/models/meshes/ee.dae" scale="1.0 1.0 1.0" />
+        <mesh filename="file://$(find canadarm_description)/models/meshes/ee.dae" scale="1.0 1.0 1.0" />
       </geometry>
     </visual>
@@ -286,5 +286,5 @@
       <origin rpy="0 -3.1415 0" xyz="0 0 0"/>
       <geometry>
-        <mesh filename="$(find canadarm_description)/models/meshes/ee.stl" scale="1.0 1.0 1.0" />
+        <mesh filename="file://$(find canadarm_description)/models/meshes/ee.stl" scale="1.0 1.0 1.0" />
       </geometry>
     </collision>
