Commit message: Rearranged objects within models forlders for easier reuse

File: ingenuity_mars_helicopter/ingenuity_description/urdf/ingenuity_description.urdf (robot description, URDF)
Before this commit: robot ingenuity_model, 8 links, 7 joints
Links:
- removed link ingenuity_model
- removed link ingenuity_model/blade_1
- removed link ingenuity_model/blade_2
- removed link ingenuity_model/blade_3
- removed link ingenuity_model/blade_4
- removed link ingenuity_model/rod_1
- removed link ingenuity_model/rod_2
- removed link ingenuity_world
- added link blade_1, mass 0.01
- added link blade_2, mass 0.01
- added link blade_3, mass 0.01
- added link blade_4, mass 0.01
- added link body, mass 10.0; visual mesh filename=package://ingenuity_description/models/ingenuity/meshes/bas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 scale=1 1 1
- added link rod_1, mass 1.0; visual mesh filename=package://ingenuity_description/models/ingenuity/meshes/rot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 scale=1 1 1
- added link rod_2, mass 1.0; visual mesh filename=package://ingenuity_description/models/ingenuity/meshes/rot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 scale=1 1 1
- added link solar_panel; visual mesh filename=package://ingenuity_description/models/ingenuity/meshes/sol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 scale=1 1 1
Joints:
- removed joint ingenuity_model/blade_1_joint
- removed joint ingenuity_model/blade_2_joint
- removed joint ingenuity_model/blade_3_joint
- removed joint ingenuity_model/blade_4_joint
- removed joint ingenuity_model/rod_1_joint
- removed joint ingenuity_model/rod_2_joint
- removed joint lift_drag_to_ingenuity_model
- added joint blade_1_joint: type fixed, parent rod_1, child blade_1, origin xyz=0.0 -0.5 0.0 rpy=0.0 0.0 0.0
- added joint blade_2_joint: type fixed, parent rod_1, child blade_2, origin xyz=0.0 0.5 0.0 rpy=0.0 0.0 0.0
- added joint blade_3_joint: type fixed, parent rod_2, child blade_3, origin xyz=0.0 0.0 0.0 rpy=0.0 0.0 0.0
- added joint blade_4_joint: type fixed, parent rod_2, child blade_4, origin xyz=0.0 0.0 0.0 rpy=0.0 0.0 0.0
- added joint rod_1_joint: type revolute, parent body, child rod_1, origin xyz=0.0 0.0 0.5 rpy=0.0 0.0 0.0, axis 0.0 0.0 -1.0, limit lower=-1e16 upper=1e16 effort=1e5 velocity=5000
- added joint rod_2_joint: type revolute, parent body, child rod_2, origin xyz=0.0 0.0 0.5 rpy=0.0 0.0 0.0, axis 0.0 0.0 1.0, limit lower=-1e16 upper=1e16 effort=1e5 velocity=5000
- added joint solar_panel_joint: type fixed, parent body, child solar_panel, origin xyz=0 0 0 rpy=0 0 0
