Commit message: Added solar panel with uniform blue color

File: lunar_pole_exploration_rover/lunar_pole_exploration_rover_gazebo/models/lunar_pole_exploration_rover/urdf/chassis.xacro (robot description, xacro)
@@ -76,12 +76,12 @@
 					rpy="0 0 0"/>
 			<geometry>
-				<mesh filename="package://lunar_pole_exploration_rover_gazebo/models/lunar_pole_exploration_rover/meshes/solar_panel.dae" scale="${scale_XYZ} ${scale_XYZ} ${scale_XYZ}"/>
-			</geometry>
-		</collision>
-		<visual>
-			<origin xyz="0 0 0"
-					rpy="0 0 0"/>
-			<geometry>
-				<mesh filename="package://lunar_pole_exploration_rover_gazebo/models/lunar_pole_exploration_rover/meshes/solar_panel.dae" scale="${scale_XYZ} ${scale_XYZ} ${scale_XYZ}"/>
+				<mesh filename="package://lunar_pole_exploration_rover_gazebo/models/lunar_pole_exploration_rover/meshes/solar_panel_dark_blue.dae" scale="${scale_XYZ} ${scale_XYZ} ${scale_XYZ}"/>
+			</geometry>
+		</collision>
+		<visual>
+			<origin xyz="0 0 0"
+					rpy="0 0 0"/>
+			<geometry>
+				<mesh filename="package://lunar_pole_exploration_rover_gazebo/models/lunar_pole_exploration_rover/meshes/solar_panel_dark_blue.dae" scale="${scale_XYZ} ${scale_XYZ} ${scale_XYZ}"/>
 			</geometry>
 		</visual>
@@ -102,12 +102,12 @@
 					rpy="0 0 0"/>
 			<geometry>
-				<mesh filename="package://lunar_pole_exploration_rover_gazebo/models/lunar_pole_exploration_rover/meshes/solar_panel.dae" scale="${scale_XYZ} ${scale_XYZ} ${scale_XYZ}"/>
-			</geometry>
-		</collision>
-		<visual>
-			<origin xyz="0 0 0"
-					rpy="0 0 0"/>
-			<geometry>
-				<mesh filename="package://lunar_pole_exploration_rover_gazebo/models/lunar_pole_exploration_rover/meshes/solar_panel.dae" scale="${scale_XYZ} ${scale_XYZ} ${scale_XYZ}"/>
+				<mesh filename="package://lunar_pole_exploration_rover_gazebo/models/lunar_pole_exploration_rover/meshes/solar_panel_dark_blue.dae" scale="${scale_XYZ} ${scale_XYZ} ${scale_XYZ}"/>
+			</geometry>
+		</collision>
+		<visual>
+			<origin xyz="0 0 0"
+					rpy="0 0 0"/>
+			<geometry>
+				<mesh filename="package://lunar_pole_exploration_rover_gazebo/models/lunar_pole_exploration_rover/meshes/solar_panel_dark_blue.dae" scale="${scale_XYZ} ${scale_XYZ} ${scale_XYZ}"/>
 			</geometry>
 		</visual>
@@ -128,12 +128,12 @@
 					rpy="0 0 0"/>
 			<geometry>
-				<mesh filename="package://lunar_pole_exploration_rover_gazebo/models/lunar_pole_exploration_rover/meshes/solar_panel.dae" scale="${scale_XYZ} ${scale_XYZ} ${scale_XYZ}"/>
-			</geometry>
-		</collision>
-		<visual>
-			<origin xyz="0 0 0"
-					rpy="0 0 0"/>
-			<geometry>
-				<mesh filename="package://lunar_pole_exploration_rover_gazebo/models/lunar_pole_exploration_rover/meshes/solar_panel.dae" scale="${scale_XYZ} ${scale_XYZ} ${scale_XYZ}"/>
+				<mesh filename="package://lunar_pole_exploration_rover_gazebo/models/lunar_pole_exploration_rover/meshes/solar_panel_dark_blue.dae" scale="${scale_XYZ} ${scale_XYZ} ${scale_XYZ}"/>
+			</geometry>
+		</collision>
+		<visual>
+			<origin xyz="0 0 0"
+					rpy="0 0 0"/>
+			<geometry>
+				<mesh filename="package://lunar_pole_exploration_rover_gazebo/models/lunar_pole_exploration_rover/meshes/solar_panel_dark_blue.dae" scale="${scale_XYZ} ${scale_XYZ} ${scale_XYZ}"/>
 			</geometry>
 		</visual>

Commit message: Sensors load

File: lunar_pole_exploration_rover/lunar_pole_exploration_rover_gazebo/models/lunar_pole_exploration_rover/urdf/chassis.xacro (robot description, xacro)
@@ -225,4 +225,96 @@
 		<origin xyz="-0.705 0.150 0.682" rpy="0 0 ${PI}"/>
 	</joint>
+	<link name="haz_camera_link_left_front">
+		<!-- Inertial for gazebo to take it into account, Put 1gr weight -->
+		<inertial>
+			<origin xyz="0 0 0" rpy="0 0 0"/>
+			<mass value="0.001" />
+			<inertia ixx="9.1875e-09" ixy="0.0" ixz="0.0" iyy="9.1875e-09" iyz="0.0" izz="1.378125e-08"/>
+		</inertial>
+		<visual>
+			<origin rpy="0.0 0 0" xyz="0 0 0"/>
+			<geometry>
+				<box size="0.0005 0.0005 0.0005"/>
+			</geometry>
+			<material name="camera_green"/>
+		</visual>
+	</link>
+	<gazebo reference="haz_camera_link_left_front">
+		<material>Gazebo/Green</material>
+	</gazebo>
+	<joint name="haz_camera_link_left_front_joint" type="fixed">
+		<parent link="body"/>
+		<child link="haz_camera_link_left_front"/>
+		<origin xyz="0.270 0.310 0.110" rpy="0 ${PI/4} ${PI/4}"/>
+	</joint>
+	<link name="haz_camera_link_left_rear">
+		<!-- Inertial for gazebo to take it into account, Put 1gr weight -->
+		<inertial>
+			<origin xyz="0 0 0" rpy="0 0 0"/>
+			<mass value="0.001" />
+			<inertia ixx="9.1875e-09" ixy="0.0" ixz="0.0" iyy="9.1875e-09" iyz="0.0" izz="1.378125e-08"/>
+		</inertial>
+		<visual>
+			<origin rpy="0.0 0 0" xyz="0 0 0"/>
+			<geometry>
+				<box size="0.0005 0.0005 0.0005"/>
+			</geometry>
+			<material name="camera_green"/>
+		</visual>
+	</link>
+	<gazebo reference="haz_camera_link_left_rear">
+		<material>Gazebo/Green</material>
+	</gazebo>
+	<joint name="haz_camera_link_left_rear_joint" type="fixed">
+		<parent link="body"/>
+		<child link="haz_camera_link_left_rear"/>
+		<origin xyz="-0.270 0.310 0.110" rpy="0 ${PI/4} ${PI/4 + PI/2}"/>
+	</joint>
+		<link name="haz_camera_link_right_front">
+		<!-- Inertial for gazebo to take it into account, Put 1gr weight -->
+		<inertial>
+			<origin xyz="0 0 0" rpy="0 0 0"/>
+			<mass value="0.001" />
+			<inertia ixx="9.1875e-09" ixy="0.0" ixz="0.0" iyy="9.1875e-09" iyz="0.0" izz="1.378125e-08"/>
+		</inertial>
+		<visual>
+			<origin rpy="0.0 0 0" xyz="0 0 0"/>
+			<geometry>
+				<box size="0.0005 0.0005 0.0005"/>
+			</geometry>
+			<material name="camera_green"/>
+		</visual>
+	</link>
+	<gazebo reference="haz_camera_link_right_front">
+		<material>Gazebo/Green</material>
+	</gazebo>
+	<joint name="haz_camera_link_right_front_joint" type="fixed">
+		<parent link="body"/>
+		<child link="haz_camera_link_right_front"/>
+		<origin xyz="0.270 -0.310 0.110" rpy="0 ${PI/4} ${-PI/4}"/>
+	</joint>
+		<link name="haz_camera_link_right_rear">
+		<!-- Inertial for gazebo to take it into account, Put 1gr weight -->
+		<inertial>
+			<origin xyz="0 0 0" rpy="0 0 0"/>
+			<mass value="0.001" />
+			<inertia ixx="9.1875e-09" ixy="0.0" ixz="0.0" iyy="9.1875e-09" iyz="0.0" izz="1.378125e-08"/>
+		</inertial>
+		<visual>
+			<origin rpy="0.0 0 0" xyz="0 0 0"/>
+			<geometry>
+				<box size="0.0005 0.0005 0.0005"/>
+			</geometry>
+			<material name="camera_green"/>
+		</visual>
+	</link>
+	<gazebo reference="haz_camera_link_right_rear">
+		<material>Gazebo/Green</material>
+	</gazebo>
+	<joint name="haz_camera_link_right_rear_joint" type="fixed">
+		<parent link="body"/>
+		<child link="haz_camera_link_right_rear"/>
+		<origin xyz="-0.270 -0.310 0.110" rpy="0 ${PI/4} ${-PI/4 - PI/2}"/>
+	</joint>
   </xacro:macro>
 </robot>

File: lunar_pole_exploration_rover/lunar_pole_exploration_rover_gazebo/models/lunar_pole_exploration_rover/urdf/wheel.xacro (robot description, xacro)
@@ -10,4 +10,12 @@
 					<cylinder radius="${wheelRadius}" length="${wheelWidth}"/>
 				</geometry>
+				<surface>
+					<friction>
+						<ode>
+							<mu>1.0</mu>
+							<mu2>1.0</mu2>
+						</ode>
+					</friction>
+				</surface>
 			</collision>
 			<visual>
@@ -29,6 +37,6 @@
 		</link>
 	  <gazebo reference="${wheel_name}">
-	    <mu1 value="1.0"/>
-	    <mu2 value="1.0"/>
+	    <!-- <mu1 value="1.0"/> -->
+	    <!-- <mu2 value="1.0"/> -->
 	    <kp  value="10000000.0" />
 	    <kd>100.0</kd>
