Commit message: disable collisions in axle and suspension because they plummet simulation speed (about 5x slower)

File: lunar_pole_exploration_rover/lunar_pole_exploration_rover_gazebo/models/lunar_pole_exploration_rover/urdf/wheel_assembly.xacro (robot description, xacro)
@@ -7,5 +7,5 @@
     <!-- tY is either 1 for ${side} side or -1 for right side -->
     <link name='${placement}_${side}_suspension'>
-        <collision>
+        <!-- <collision>
           <origin xyz="0 0 0"
               rpy="0 0 0"/>
@@ -13,5 +13,5 @@
             <mesh filename="package://lunar_pole_exploration_rover_gazebo/models/lunar_pole_exploration_rover/meshes/suspension_${side}.dae" scale="${scale_XYZ} ${scale_XYZ} ${scale_XYZ}"/>
           </geometry>
-        </collision>
+        </collision> -->
         <visual>
           <origin xyz="0 0 0"
@@ -42,5 +42,5 @@
       </joint>
       <link name='${placement}_${side}_wheel_axle'>
-        <collision>
+        <!-- <collision>
           <origin xyz="0 0 0"
               rpy="0 0 0"/>
@@ -48,5 +48,5 @@
             <mesh filename="package://lunar_pole_exploration_rover_gazebo/models/lunar_pole_exploration_rover/meshes/wheel_axle_${side}.dae" scale="${scale_XYZ} ${scale_XYZ} ${scale_XYZ}"/>
           </geometry>
-        </collision>
+        </collision> -->
         <visual>
           <origin xyz="0 0 0"
